File: hardware/kicad/LIS3MDL.kicad_sch (KiCad schematic)
At the start: 7 parts, among them U2 LIS2MDLTR

Commit message: Moved sensors from stamp to direct placement
Parts:
- removed J201: (no value), footprints:Stamp, symbol rollercoasterometer2026:STAMP
