File: hardware/kicad/RP2354.kicad_pcb (KiCad board)
At the start: 2 copper layers, 52 x 51 mm, 28 parts, among them U501 RP2350_60QFN, Y501 ABM8-272-T3

Commit message: Import rp2354 module
Parts:
- removed H1, H2, H3, H4: MountingHole, MountingHole:MountingHole_2.7mm_M2.5
- renumbered R6 to R560
Routing:
- net /GPIO0: track 39.0 -> 0.00 mm, vias 2 -> 0
- net /GPIO29_ADC3: track 33.6 -> 0.00 mm
- net /GPIO28_ADC2: track 31.9 -> 0.00 mm
- net /GPIO27_ADC1: track 30.3 -> 0.00 mm
- net /GPIO1: track 29.8 -> 0.00 mm
- net /GPIO26_ADC0: track 28.6 -> 0.00 mm
- net /GPIO2: track 28.2 -> 0.00 mm
- net /SWCLK: track 27.8 -> 0.00 mm
- net /GPIO25: track 27.7 -> 0.00 mm
- net GND: track 37.5 -> 9.83 mm, vias 27 -> 17
- net /GPIO3: track 26.5 -> 0.00 mm
- net /GPIO24: track 26.1 -> 0.00 mm
- net /SWD: track 25.4 -> 0.00 mm
- net /GPIO15: track 25.2 -> 0.00 mm
- net /GPIO4: track 25.0 -> 0.00 mm
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- removed copper zone on B.Cu, net GND
- removed copper zone on F.Cu, net VBUS
Other:
- board outline removed
- board text removed: "3V3"
- board text removed: "ADC 26-29"
- board text removed: "DEBUG"
- board text removed: "GND"
- board text removed: "GP0"
- board text removed: "GP1"
- board text removed: "GP10"
- board text removed: "GP11"
- board text removed: "GP12"
- board text removed: "GP13"
- board text removed: "GP14"
- board text removed: "GP15"
- board text removed: "GP16"
- board text removed: "GP17"
- board text removed: "GP18"
- board text removed: "GP19"
- board text removed: "GP2"
- board text removed: "GP20"
- board text removed: "GP21"
- board text removed: "GP22"
- board text removed: "GP23"
- board text removed: "GP24"
- board text removed: "GP25"
- board text removed: "GP26"
- board text removed: "GP27"
- board text removed: "GP28"
- board text removed: "GP29"
- board text removed: "GP3"
- board text removed: "GP4"
- board text removed: "GP5"
- board text removed: "GP6"
- board text removed: "GP7"
- board text removed: "GP8"
- board text removed: "GP9"
- board text removed: "Minimal Design Example REV3"
- board text removed: "Outer Row GND"
- board text removed: "RUN"
- board text removed: "Raspberry Pi RP2350A QFN-60"
- board text removed: "SWCLK"
- board text removed: "SWD"
