File: hardware/kicad/RP2354.kicad_sch (KiCad schematic)
At the start: 24 parts, among them U4 RP2354A, Y501 ABM8-272-T3

Commit message: Import rp2354 module
Parts:
- C549, C550: footprint RP2350_60QFN_minimal:C_0402_1005Metric_small_pads -> footprints:C_0402_1005Metric_small_pads
- L550: footprint RP2350_60QFN_minimal:L_pol_2016 -> footprints:L_pol_2016
- U501: renamed from U4; footprint RP2350_60QFN_minimal:RP2350-QFN-60-1EP_7x7_P0.4mm_EP3.4x3.4mm_ThermalVias -> footprints:RP2350-QFN-60-1EP_7x7_P0.4mm_EP3.4x3.4mm_ThermalVias
Connections:
- net USB_D-: now also R551.1
- net USB_D++: now reaches R552.2, U501.52 (USB_DP)
- net USB_D--: now reaches R551.2, U501.51 (USB_DM)
